Commit message: fix(nav): improve Lite3 obstacle avoidance responsiveness
Use low-latency chassis odometry for Nav2 while keeping ICP localization in a private frame and bridging its global correction.

Remove scan deskew latency from the navigation path, correct the MID-360 mount offset, and tune DWB, costmaps, velocity smoothing, and the 0.35 m/s safety envelope.

File: urdf/Lite3.urdf (robot description, URDF)
Before this commit: robot Lite3, 31 links, 30 joints
Joints:
- joint base_to_livox: origin xyz=0 0 0.10 rpy=0 0 0 -> xyz=0.045 0 0.10 rpy=0 0 0

Commit message: fix(urdf): keep mesh assets within URDF directory

File: urdf/Lite3.urdf (robot description, URDF)
Before this commit: robot Lite3, 31 links, 30 joints
Links:
- link FL_HIP: geometry collision cylinder length=0.15 radius=0.04; visual mesh filename=meshes/hip.STL scale=1 1 1
- link FL_SHANK: geometry collision cylinder length=0.10 radius=0.015; collision cylinder length=0.12 radius=0.015
- link FL_THIGH: geometry collision box size=0.04 0.045 0.2; visual mesh filename=meshes/thigh.STL
- link FR_HIP: geometry collision cylinder length=0.15 radius=0.04; visual mesh filename=meshes/hip.STL scale=1 -1 1
- link FR_SHANK: geometry collision cylinder length=0.10 radius=0.015; collision cylinder length=0.12 radius=0.015
- link FR_THIGH: geometry collision box size=0.04 0.045 0.2; visual mesh filename=meshes/thigh.STL scale=1 -1 1
- link HL_HIP: geometry collision cylinder length=0.15 radius=0.04; visual mesh filename=meshes/hip.STL scale=-1 1 1
- link HL_SHANK: geometry collision cylinder length=0.10 radius=0.015; collision cylinder length=0.12 radius=0.015
- link HL_THIGH: geometry collision box size=0.04 0.045 0.2; visual mesh filename=meshes/thigh.STL
- link HR_HIP: geometry collision cylinder length=0.15 radius=0.04; visual mesh filename=meshes/hip.STL scale=-1 -1 1
- link HR_SHANK: geometry collision cylinder length=0.10 radius=0.015; collision cylinder length=0.12 radius=0.015
- link HR_THIGH: geometry collision box size=0.04 0.045 0.2; visual mesh filename=meshes/thigh.STL scale=1 -1 1
- link TORSO: geometry collision box size=0.25 0.2 0.12; collision box size=0.5 0.1 0.12
